File: Generator/generator.sch (EAGLE design)
At the start: 28 parts, among them IC2 317EMP, X1 22-23-2021

Commit message: test
Parts:
- added C12: 10uF, rcl:C-EUC0805
- added JP1, JP2, JP3, JP4, JP5, JP6, JP7, JP8, JP9: (no value), pinhead:PINHD-1X1
- renumbered IC1 to XR2206CP
Connections:
- net GND: now also C12.2, JP3.1
- net N$11: now also C12.1
- net SIN_TRI: now also JP1.1
- net SQR: now also JP2.1
Changed lines of the file:
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@@
 <?xml version="1.0" encoding="utf-8"?>
 <!DOCTYPE eagle SYSTEM "eagle.dtd">
-<eagle version="7.2.0">
+<eagle version="7.3.0">
 <drawing>
 <settings>
@@
 <part name="C8" library="rcl" deviceset="C-EU" device="C0805" value="100nF"/>
 <part name="C9" library="rcl" deviceset="C-EU" device="C0805" value="100pF"/>
-<part name="IC1" library="exar" deviceset="XR-2206" device=""/>
+<part name="XR2206CP" library="exar" deviceset="XR-2206" device=""/>
 <part name="R1" library="rcl" deviceset="R-EU_" device="R0805" value="10k"/>
 <part name="S2" library="switch" deviceset="ELMA-01-1X6" device=""/>
@@
 <part name="GND10" library="supply1" deviceset="GND" device=""/>
 <part name="R11" library="rcl" deviceset="R-EU_" device="R0805" value="1k"/>
+<part name="JP1" library="pinhead" deviceset="PINHD-1X1" device=""/>
+<part name="JP2" library="pinhead" deviceset="PINHD-1X1" device=""/>
+<part name="JP3" library="pinhead" deviceset="PINHD-1X1" device=""/>
+<part name="JP4" library="pinhead" deviceset="PINHD-1X1" device=""/>
+<part name="JP5" library="pinhead" deviceset="PINHD-1X1" device=""/>
+<part name="JP6" library="pinhead" deviceset="PINHD-1X1" device=""/>
+<part name="JP7" library="pinhead" deviceset="PINHD-1X1" device=""/>
+<part name="JP8" library="pinhead" deviceset="PINHD-1X1" device=""/>
+<part name="JP9" library="pinhead" deviceset="PINHD-1X1" device=""/>
+<part name="C12" library="rcl" deviceset="C-EU" device="C0805" value="10uF"/>
 </parts>
 <sheets>
@@
 <instance part="C8" gate="G$1" x="-12.7" y="22.86" rot="R90"/>
 <instance part="C9" gate="G$1" x="-12.7" y="-2.54" rot="R90"/>
-<instance part="IC1" gate="G$1" x="76.2" y="40.64"/>
+<instance part="XR2206CP" gate="G$1" x="76.2" y="40.64"/>
 <instance part="R1" gate="G$1" x="17.78" y="58.42"/>
 <instance part="S2" gate="G$1" x="17.78" y="35.56" rot="R270"/>
@@
 <instance part="GND10" gate="1" x="243.84" y="-15.24"/>
 <instance part="R11" gate="G$1" x="243.84" y="12.7" rot="R90"/>
+<instance part="JP1" gate="G$1" x="147.32" y="83.82" rot="R90"/>
+<instance part="JP2" gate="G$1" x="152.4" y="83.82" rot="R90"/>
+<instance part="JP3" gate="G$1" x="157.48" y="83.82" rot="R90"/>
+<instance part="JP4" gate="G$1" x="71.12" y="-45.72" rot="R90"/>
+<instance part="JP5" gate="G$1" x="76.2" y="-45.72" rot="R90"/>
+<instance part="JP6" gate="G$1" x="81.28" y="-45.72" rot="R90"/>
+<instance part="JP7" gate="G$1" x="86.36" y="-45.72" rot="R90"/>
+<instance part="JP8" gate="G$1" x="91.44" y="-45.72" rot="R90"/>
+<instance part="JP9" gate="G$1" x="96.52" y="-45.72" rot="R90"/>
+<instance part="C12" gate="G$1" x="104.14" y="25.4"/>
 </instances>
 <busses>
@@
 <wire x1="25.4" y1="40.64" x2="30.48" y2="40.64" width="0.1524" layer="91"/>
 <wire x1="30.48" y1="40.64" x2="30.48" y2="30.48" width="0.1524" layer="91"/>
-<pinref part="IC1" gate="G$1" pin="C1"/>
+<pinref part="XR2206CP" gate="G$1" pin="C1"/>
 <wire x1="30.48" y1="30.48" x2="58.42" y2="30.48" width="0.1524" layer="91"/>
 <pinref part="S2" gate="G$1" pin="S"/>
@@
 <net name="C2" class="0">
 <segment>
-<pinref part="IC1" gate="G$1" pin="C2"/>
+<pinref part="XR2206CP" gate="G$1" pin="C2"/>
 <wire x1="58.42" y1="27.94" x2="35.56" y2="27.94" width="0.1524" layer="91"/>
 <label x="35.56" y="27.94" size="1.27" layer="95" rot="R180" xref="yes"/>
@@
 <wire x1="35.56" y1="58.42" x2="35.56" y2="35.56" width="0.1524" layer="91"/>
 <wire x1="35.56" y1="35.56" x2="58.42" y2="35.56" width="0.1524" layer="91"/>
-<pinref part="IC1" gate="G$1" pin="R1"/>
+<pinref part="XR2206CP" gate="G$1" pin="R1"/>
 </segment>
 </net>
@@
 <pinref part="GND2" gate="1" pin="GND"/>
 <wire x1="45.72" y1="63.5" x2="45.72" y2="66.04" width="0.1524" layer="91"/>
-<pinref part="IC1" gate="G$1" pin="AM_IN"/>
+<pinref part="XR2206CP" gate="G$1" pin="AM_IN"/>
 <wire x1="45.72" y1="66.04" x2="45.72" y2="71.12" width="0.1524" layer="91"/>
 <wire x1="58.42" y1="53.34" x2="53.34" y2="53.34" width="0.1524" layer="91"/>
@@
 <pinref part="R7" gate="G$1" pin="1"/>
 <wire x1="104.14" y1="17.78" x2="106.68" y2="17.78" width="0.1524" layer="91"/>
+<pinref part="C12" gate="G$1" pin="2"/>
+<wire x1="104.14" y1="20.32" x2="104.14" y2="17.78" width="0.1524" layer="91"/>
+<junction x="104.14" y="17.78"/>
 </segment>
 <segment>
@@
 <wire x1="243.84" y1="-12.7" x2="243.84" y2="-2.54" width="0.1524" layer="91"/>
 </segment>
+<segment>
+<pinref part="JP3" gate="G$1" pin="1"/>
+<wire x1="157.48" y1="81.28" x2="157.48" y2="71.12" width="0.1524" layer="91"/>
+<label x="157.48" y="71.12" size="1.27" layer="95" rot="R270" xref="yes"/>
+</segment>
 </net>
 <net name="N$10" class="0">
 <segment>
-<pinref part="IC1" gate="G$1" pin="BYPASS"/>
+<pinref part="XR2206CP" gate="G$1" pin="BYPASS"/>
 <wire x1="58.42" y1="48.26" x2="38.1" y2="48.26" width="0.1524" layer="91"/>
 <pinref part="C1" gate="G$1" pin="2"/>
@@
 <net name="SQR" class="0">
 <segment>
-<pinref part="IC1" gate="G$1" pin="SYNC"/>
+<pinref part="XR2206CP" gate="G$1" pin="SYNC"/>
 <pinref part="R3" gate="G$1" pin="1"/>
 <wire x1="93.98" y1="48.26" x2="99.06" y2="48.26" width="0.1524" layer="91"/>
@@
 <wire x1="99.06" y1="50.8" x2="101.6" y2="50.8" width="0.1524" layer="91"/>
 <label x="101.6" y="50.8" size="1.27" layer="95" xref="yes"/>
+</segment>
+<segment>
+<pinref part="JP2" gate="G$1" pin="1"/>
+<wire x1="152.4" y1="81.28" x2="152.4" y2="71.12" width="0.1524" layer="91"/>
+<label x="152.4" y="71.12" size="1.27" layer="95" rot="R270" xref="yes"/>
 </segment>
 </net>
@@
 <pinref part="R4" gate="1" pin="A"/>
 <wire x1="53.34" y1="20.32" x2="53.34" y2="38.1" width="0.1524" layer="91"/>
-<pinref part="IC1" gate="G$1" pin="S_ADJ@2"/>
+<pinref part="XR2206CP" gate="G$1" pin="S_ADJ@2"/>
 <wire x1="53.34" y1="38.1" x2="58.42" y2="38.1" width="0.1524" layer="91"/>
 </segment>
@@
 <wire x1="43.18" y1="22.86" x2="50.8" y2="22.86" width="0.1524" layer="91"/>
 <wire x1="50.8" y1="22.86" x2="50.8" y2="40.64" width="0.1524" layer="91"/>
-<pinref part="IC1" gate="G$1" pin="S_ADJ@1"/>
+<pinref part="XR2206CP" gate="G$1" pin="S_ADJ@1"/>
 <wire x1="50.8" y1="40.64" x2="58.42" y2="40.64" width="0.1524" layer="91"/>
 </segment>
@@
 <net name="N$14" class="0">
 <segment>
-<pinref part="IC1" gate="G$1" pin="W_ADJ@1"/>
+<pinref part="XR2206CP" gate="G$1" pin="W_ADJ@1"/>
 <wire x1="58.42" y1="45.72" x2="38.1" y2="45.72" width="0.1524" layer="91"/>
 <wire x1="38.1" y1="45.72" x2="38.1" y2="17.78" width="0.1524" layer="91"/>
@@
 <net name="N$15" class="0">
 <segment>
-<pinref part="IC1" gate="G$1" pin="W_ADJ@2"/>
+<pinref part="XR2206CP" gate="G$1" pin="W_ADJ@2"/>
 <wire x1="58.42" y1="43.18" x2="40.64" y2="43.18" width="0.1524" layer="91"/>
 <wire x1="40.64" y1="43.18" x2="40.64" y2="15.24" width="0.1524" layer="91"/>
@@
 <net name="SIN_TRI" class="0">
 <segment>
-<pinref part="IC1" gate="G$1" pin="SI/TR"/>
+<pinref part="XR2206CP" gate="G$1" pin="SI/TR"/>
 <wire x1="93.98" y1="53.34" x2="101.6" y2="53.34" width="0.1524" layer="91"/>
 <label x="101.6" y="53.34" size="1.27" layer="95" xref="yes"/>
+</segment>
+<segment>
+<pinref part="JP1" gate="G$1" pin="1"/>
+<wire x1="147.32" y1="81.28" x2="147.32" y2="71.12" width="0.1524" layer="91"/>
+<label x="147.32" y="71.12" size="1.27" layer="95" rot="R270" xref="yes"/>
 </segment>
 </net>
@@
 <wire x1="111.76" y1="22.86" x2="119.38" y2="22.86" width="0.1524" layer="91"/>
 <junction x="119.38" y="22.86"/>
+<pinref part="C12" gate="G$1" pin="1"/>
+<wire x1="104.14" y1="27.94" x2="104.14" y2="30.48" width="0.1524" layer="91"/>
+<wire x1="104.14" y1="30.48" x2="111.76" y2="30.48" width="0.1524" layer="91"/>
+<junction x="111.76" y="30.48"/>
 </segment>
 </net>
@@
 <wire x1="119.38" y1="43.18" x2="96.52" y2="43.18" width="0.1524" layer="91"/>
 <wire x1="96.52" y1="43.18" x2="96.52" y2="50.8" width="0.1524" layer="91"/>
-<pinref part="IC1" gate="G$1" pin="MULT_OUT"/>
+<pinref part="XR2206CP" gate="G$1" pin="MULT_OUT"/>
 <wire x1="96.52" y1="50.8" x2="93.98" y2="50.8" width="0.1524" layer="91"/>
 </segment>
